File: docs/kicad/uno_display_connector/uno_display_connector.sch (KiCad schematic (older format))
At the start: 3 parts, among them J1 Conn_01x08, J2 Conn_01x08, U1 uno_display

Commit message: start MAKE NEW motherboard and display_connector FOR olds TeensyExprssion box with TE2 code
Connections:
- net +3V3: now also J2.1 (Pin_1); no longer J2.2 (Pin_2)
- net +5V: now also J2.2 (Pin_2); no longer J2.1 (Pin_1)
Changed lines of the file:
@@
 L power:+5V #PWR06
 U 1 1 64E16798
+P 3350 4700
+F 0 "#PWR06" H 3350 4550 50  0001 C CNN
+F 1 "+5V" V 3350 4850 50  0000 L CNN
+F 2 "" H 3350 4700 50  0001 C CNN
+F 3 "" H 3350 4700 50  0001 C CNN
+	1    3350 4700
+	0    1    1    0
+$EndComp
+$Comp
+L power:+3V3 #PWR05
+U 1 1 64E32F64
 P 3350 4800
-F 0 "#PWR06" H 3350 4650 50  0001 C CNN
-F 1 "+5V" V 3350 4950 50  0000 L CNN
+F 0 "#PWR05" H 3350 4650 50  0001 C CNN
+F 1 "+3V3" V 3350 5050 50  0000 C CNN
 F 2 "" H 3350 4800 50  0001 C CNN
 F 3 "" H 3350 4800 50  0001 C CNN
@@
 	0    1    1    0
 $EndComp
-$Comp
-L power:+3V3 #PWR05
-U 1 1 64E32F64
-P 3350 4700
-F 0 "#PWR05" H 3350 4550 50  0001 C CNN
-F 1 "+3V3" V 3350 4950 50  0000 C CNN
-F 2 "" H 3350 4700 50  0001 C CNN
-F 3 "" H 3350 4700 50  0001 C CNN
-	1    3350 4700
-	0    1    1    0
-$EndComp

Commit message: kicad - corrected TFT data pin order for new teensyExpression2 board/code
Other:
- note added: "NOTE that LCD_D0 and LCD_D1 are switched\nwhile soldering the wires onto this connector so \nALL DATA LINES COME OUT IN ORDER on the\nother end as REQUIRED by the mother board!!!"
Changed lines of the file:
@@
 	0    1    1    0
 $EndComp
+Text Notes 1200 3000 0    50   ~ 0
+NOTE that LCD_D0 and LCD_D1 are switched\nwhile soldering the wires onto this connector so  \nALL DATA LINES COME OUT IN ORDER on the\nother end as REQUIRED by the mother board!!!
 $EndSCHEMATC

Commit message: BUILD new combined mother_board and uno_display_connector. PRINT new display_frame.
Parts:
- J1, J2: footprint cnc3018-PCB:my8Pin -> 0_my_footprints:my8Pin
Changed lines of the file:
@@
 F 0 "J1" H 3118 2325 50  0000 C CNN
 F 1 "Conn_01x08" H 3118 2416 50  0000 C CNN
-F 2 "cnc3018-PCB:my8Pin" H 3200 2950 50  0001 C CNN
+F 2 "0_my_footprints:my8Pin" H 3200 2950 50  0001 C CNN
 F 3 "~" H 3200 2950 50  0001 C CNN
 	1    3200 2950
@@
 F 0 "J2" H 3068 3875 50  0000 C CNN
 F 1 "Conn_01x08" H 3068 3966 50  0000 C CNN
-F 2 "cnc3018-PCB:my8Pin" H 3150 4500 50  0001 C CNN
+F 2 "0_my_footprints:my8Pin" H 3150 4500 50  0001 C CNN
 F 3 "~" H 3150 4500 50  0001 C CNN
 	1    3150 4500

Commit message: AFTER BUILD NEW PCBs - corrected display connector pins; removed old combined plot and gcode file
Connections:
- net +3V3: now also J2.2 (Pin_2); no longer J2.1 (Pin_1)
- net +5V: now also J2.1 (Pin_1); no longer J2.2 (Pin_2)
Changed lines of the file:
@@
 L power:+5V #PWR06
 U 1 1 64E16798
+P 3350 4800
+F 0 "#PWR06" H 3350 4650 50  0001 C CNN
+F 1 "+5V" V 3350 4950 50  0000 L CNN
+F 2 "" H 3350 4800 50  0001 C CNN
+F 3 "" H 3350 4800 50  0001 C CNN
+	1    3350 4800
+	0    1    1    0
+$EndComp
+$Comp
+L power:+3V3 #PWR05
+U 1 1 64E32F64
 P 3350 4700
-F 0 "#PWR06" H 3350 4550 50  0001 C CNN
-F 1 "+5V" V 3350 4850 50  0000 L CNN
+F 0 "#PWR05" H 3350 4550 50  0001 C CNN
+F 1 "+3V3" V 3350 4950 50  0000 C CNN
 F 2 "" H 3350 4700 50  0001 C CNN
 F 3 "" H 3350 4700 50  0001 C CNN
@@
 	0    1    1    0
 $EndComp
-$Comp
-L power:+3V3 #PWR05
-U 1 1 64E32F64
-P 3350 4800
-F 0 "#PWR05" H 3350 4650 50  0001 C CNN
-F 1 "+3V3" V 3350 5050 50  0000 C CNN
-F 2 "" H 3350 4800 50  0001 C CNN
-F 3 "" H 3350 4800 50  0001 C CNN
-	1    3350 4800
-	0    1    1    0
-$EndComp
