File: docs/kicad/serial_connector/serial_connector.sch (KiCad schematic (older format))
At the start: 2 parts

Commit message: AFTER TE2 REBUILD - new gcode for left, top, and back.  Corrected symbols for Serial Connector (and on motherboard)
Parts:
- removed J?: JACK, symbol Connector:AudioJack2_Ground
- added J?: myAudioJack3.5mm, symbol 0_my_symbols:myAudioJack3.5mm
Other:
- note added: "GND - SLEEVE"
- note added: "TEENSY RX2 - RING"
- note added: "TEENSY TX2 - TIP"
- note removed: "GND"
- note removed: "TEENSY RX2"
- note removed: "TEENSY TX2"
